Commit message: tool0 frame and joint adapted for bumper sensor

File: ur_description/urdf/ur.gazebo.xacro (robot description, xacro)
@@ -2,5 +2,19 @@
 <robot xmlns:xacro="http://ros.org/wiki/xacro">
   <xacro:macro name="ur_arm_gazebo" params="prefix">
-    <!-- nothing to do here at the moment -->
+    <!--gazebo reference="${prefix}ee_link">
+      <self_collide>false</self_collide>
+      <sensor name='${prefix}ee_link_sensor' type='contact'>
+        <always_on>true</always_on>
+        <update_rate>100.0</update_rate>
+        <contact>
+          <collision>${prefix}ee_link_collision</collision>
+          <topic>${prefix}ee_link_bumper</topic>
+        </contact>
+        <plugin name="${prefix}ee_link_gazebo_ros_bumper_controller" filename="libgazebo_ros_bumper.so">
+          <bodyName>${prefix}ee_link</bodyName>
+          <bumperTopicName>${prefix}ee_link_bumper</bumperTopicName>
+        </plugin>
+      </sensor>
+    </gazebo-->
   </xacro:macro>
 </robot>

File: ur_description/urdf/ur.transmission.xacro (robot description, xacro)
@@ -62,4 +62,14 @@
       </actuator>
     </transmission>
+    <transmission name="${prefix}ee_fixed_trans">
+      <type>transmission_interface/SimpleTransmission</type>
+      <joint name="${prefix}ee_fixed_joint">
+        <hardwareInterface>PositionJointInterface</hardwareInterface>
+        <hardwareInterface>VelocityJointInterface</hardwareInterface>
+      </joint>
+      <actuator name="${prefix}ee_fixed_motor">
+        <mechanicalReduction>1</mechanicalReduction>
+      </actuator>
+    </transmission>
   </xacro:macro>
 </robot>

File: ur_description/urdf/ur10.urdf.xacro (robot description, xacro)
@@ -268,4 +268,11 @@
       <child link = "${prefix}ee_link" />
       <origin xyz="0.0 ${wrist_3_length} 0.0" rpy="0.0 0.0 ${pi/2.0}" />
+      <xacro:unless value="${joint_limited}">
+        <limit lower="${-2.0 * pi}" upper="${2.0 * pi}" effort="54.0" velocity="3.2"/>
+      </xacro:unless>
+      <xacro:if value="${joint_limited}">
+        <limit lower="${wrist_3_lower_limit}" upper="${wrist_3_upper_limit}" effort="54.0" velocity="3.2"/>
+      </xacro:if>
+      <dynamics damping="0.0" friction="0.0"/>
     </joint>
     <link name="${prefix}ee_link">
@@ -291,9 +298,23 @@
     </joint>
     <!-- Frame coincident with all-zeros TCP on UR controller -->
-    <link name="${prefix}tool0"/>
+    <link name="${prefix}tool0">
+      <collision>
+        <geometry>
+          <box size="0.01 0.01 0.01"/>
+        </geometry>
+        <origin rpy="0 0 0" xyz="-0.01 0 0"/>
+      </collision>
+    </link>
     <joint name="${prefix}wrist_3_link-tool0_fixed_joint" type="fixed">
-      <origin xyz="0 ${wrist_3_length} 0" rpy="${pi/-2.0} 0 0"/>
+      <origin xyz="0.0 0.2922 0.0" rpy="0.0 0.0 ${pi/2.0}" />
       <parent link="${prefix}wrist_3_link"/>
       <child link="${prefix}tool0"/>
+      <xacro:unless value="${joint_limited}">
+        <limit lower="${-2.0 * pi}" upper="${2.0 * pi}" effort="54.0" velocity="3.2"/>
+      </xacro:unless>
+      <xacro:if value="${joint_limited}">
+        <limit lower="${wrist_3_lower_limit}" upper="${wrist_3_upper_limit}" effort="54.0" velocity="3.2"/>
+      </xacro:if>
+      <dynamics damping="0.0" friction="0.0"/>
     </joint>
   </xacro:macro>
